Commit message: update

File: ros2_ws/src/multi_sensor_perception/urdf/robot.urdf.xacro (robot description, xacro)
@@ -16,22 +16,22 @@
   <link name="base_link">
     <visual>
-      <origin xyz="0 0 0.05" rpy="0 0 0"/>
+      <origin xyz="0 0 0.06" rpy="0 0 0"/>
       <geometry>
-        <box size="0.4 0.3 0.1"/>
+        <box size="0.5 0.35 0.12"/>
       </geometry>
-      <material name="grey">
-        <color rgba="0.5 0.5 0.55 1"/>
+      <material name="blue">
+        <color rgba="0.15 0.45 0.9 1"/>
       </material>
     </visual>
     <collision>
-      <origin xyz="0 0 0.05" rpy="0 0 0"/>
+      <origin xyz="0 0 0.06" rpy="0 0 0"/>
       <geometry>
-        <box size="0.4 0.3 0.1"/>
+        <box size="0.5 0.35 0.12"/>
       </geometry>
     </collision>
     <inertial>
-      <origin xyz="0 0 0.05" rpy="0 0 0"/>
-      <mass value="5.0"/>
-      <inertia ixx="0.05" ixy="0" ixz="0" iyy="0.05" iyz="0" izz="0.05"/>
+      <origin xyz="0 0 0.06" rpy="0 0 0"/>
+      <mass value="6.0"/>
+      <inertia ixx="0.08" ixy="0" ixz="0" iyy="0.08" iyz="0" izz="0.08"/>
     </inertial>
   </link>
@@ -58,5 +58,5 @@
     <parent link="base_link"/>
     <child link="lidar_link"/>
-    <origin xyz="0 0 0.12" rpy="0 0 0"/>
+    <origin xyz="0 0 0.14" rpy="0 0 0"/>
   </joint>
   <link name="camera_link">
@@ -82,5 +82,5 @@
     <parent link="base_link"/>
     <child link="camera_link"/>
-    <origin xyz="0.22 0 0.08" rpy="0 0 0"/>
+    <origin xyz="0.27 0 0.10" rpy="0 0 0"/>
   </joint>
   <!-- Gazebo Sim sensors: explicit gz topics for simple ros_gz_bridge mapping. -->
